Commit message: fixed joints

File: urdf/rover_front_right_wheel.xacro (robot description, xacro)
@@ -52,5 +52,5 @@
 		<origin xyz="0.0599999999999999 -0.1135 -0.024" rpy="0 0 0" />
 		<parent link="base_link" />
-		<child link="rover_front_right_wheel" />
+		<child link="front_right_wheel" />
 		<axis xyz="0 1 0" />
 	</joint>

File: urdf/rover_rear_left_wheel.xacro (robot description, xacro)
@@ -52,5 +52,5 @@
 	    	<origin xyz="-0.0599999999999999 0.1135 -0.0240000000000001" rpy="0 0 0" />
 	    	<parent link="base_link" />
-	    	<child link="rover_rear_left_wheel" />
+	    	<child link="rear_left_wheel" />
 	    	<axis xyz="0 -1 0" />
 	</joint>

File: urdf/rover_rear_right_wheel.xacro (robot description, xacro)
@@ -52,5 +52,5 @@
 	    <origin xyz="-0.0600000000000001 -0.1135 -0.024" rpy="0 0 0" />
 	    <parent link="base_link" />
-	    <child link="rover_rear_right_wheel" />
+	    <child link="rear_right_wheel" />
 	    <axis xyz="0 1 0" />
 	</joint>

Commit message: wheels xacro fixed v2

File: urdf/rover_front_right_wheel.xacro (robot description, xacro)
@@ -51,5 +51,5 @@
 	<joint name="front_right_wheel_to_base" type="continuous">
 		<origin xyz="0.0599999999999999 -0.1135 -0.024" rpy="0 0 0" />
-		<parent link="base_link" />
+		<parent link="rover_base" />
 		<child link="front_right_wheel" />
 		<axis xyz="0 1 0" />

File: urdf/rover_rear_left_wheel.xacro (robot description, xacro)
@@ -51,5 +51,5 @@
 	<joint name="rear_left_wheel_to_base" type="continuous">
 	    	<origin xyz="-0.0599999999999999 0.1135 -0.0240000000000001" rpy="0 0 0" />
-	    	<parent link="base_link" />
+	    	<parent link="rover_base" />
 	    	<child link="rear_left_wheel" />
 	    	<axis xyz="0 -1 0" />
