Commit message: wheels radius added

File: urdf/rover.xacro (robot description, xacro)
@@ -2,4 +2,9 @@
 <robot name="rover" xmlns:xacro="http://www.ros.org/wiki/xacro">
 	<xacro:property name="clearance" value="0.074" />
+	<xacro:property name="wheel_radius" value="0.0485"/>
+	<xacro:property name="wheel_separation_x" value="0.128"/>
+	<xacro:property name="wheel_separation_y" value="0.128"/>
+	<xacro:property name="wheel_width" value="0.0447"/>
+	<xacro:property name="PI" value="3.1415926"/>
 	<link name="base_link">
 		<inertial>

File: urdf/rover_front_left_wheel.xacro (robot description, xacro)
@@ -29,8 +29,28 @@
     		</collision>
   	</link>
+	<link name="front_left_wheel">
+		<visual>
+			<origin xyz="0 0 0" rpy="${PI/2} 0 0" />
+			<geometry>
+				<cylinder length="${wheel_width}" radius="${wheel_radius}"/>
+			</geometry>
+			<material name="Green" />
+		</visual>
+		<collision>
+			<origin xyz="0 0 0" rpy="${PI/2} 0 0" />
+			<geometry>
+				<cylinder length="${wheel_width}" radius="${wheel_radius}"/>
+			</geometry>
+		</collision>
+	</link>
+	<joint name="front_left_wheel_to_rover_front_left_wheel" type="fixed">
+		<origin xyz="0 0 0" rpy="0 0 0" />
+		<parent link="front_left_wheel" />
+		<child link="rover_front_left_wheel" />
+	</joint>
 	<joint name="front_left_wheel_to_base" type="continuous">
 	    	<origin xyz="0.0599999999999999 0.1135 -0.024" rpy="0 0 0" />
 	    	<parent link="base_link" />
-	    	<child link="rover_front_left_wheel" />
+	    	<child link="front_left_wheel" />
 	    	<axis xyz="0 -1 0" />
 	</joint>

File: urdf/rover_front_right_wheel.xacro (robot description, xacro)
@@ -29,4 +29,24 @@
 		</collision>
 	</link>
+	<link name="front_right_wheel">
+		<visual>
+			<origin xyz="0 0 0" rpy="${PI/2} 0 0" />
+			<geometry>
+				<cylinder length="${wheel_width}" radius="${wheel_radius}"/>
+			</geometry>
+			<material name="Green" />
+		</visual>
+		<collision>
+			<origin xyz="0 0 0" rpy="${PI/2} 0 0" />
+			<geometry>
+				<cylinder length="${wheel_width}" radius="${wheel_radius}"/>
+			</geometry>
+		</collision>
+	</link>
+	<joint name="front_right_wheel_to_rover_front_right_wheel" type="fixed">
+		<origin xyz="0 0 0" rpy="0 0 0" />
+		<parent link="front_right_wheel" />
+		<child link="rover_front_right_wheel" />
+	</joint>
 	<joint name="front_right_wheel_to_base" type="continuous">
 		<origin xyz="0.0599999999999999 -0.1135 -0.024" rpy="0 0 0" />

File: urdf/rover_rear_left_wheel.xacro (robot description, xacro)
@@ -29,4 +29,24 @@
 	    	</collision>
 	</link>
+	<link name="rear_left_wheel">
+		<visual>
+			<origin xyz="0 0 0" rpy="${PI/2} 0 0" />
+			<geometry>
+				<cylinder length="${wheel_width}" radius="${wheel_radius}"/>
+			</geometry>
+			<material name="Green" />
+		</visual>
+		<collision>
+			<origin xyz="0 0 0" rpy="${PI/2} 0 0" />
+			<geometry>
+				<cylinder length="${wheel_width}" radius="${wheel_radius}"/>
+			</geometry>
+		</collision>
+	</link>
+	<joint name="rear_left_wheel_to_rover_rear_left_wheel" type="fixed">
+		<origin xyz="0 0 0" rpy="0 0 0" />
+		<parent link="rear_left_wheel" />
+		<child link="rover_rear_left_wheel" />
+	</joint>
 	<joint name="rear_left_wheel_to_base" type="continuous">
 	    	<origin xyz="-0.0599999999999999 0.1135 -0.0240000000000001" rpy="0 0 0" />

File: urdf/rover_rear_right_wheel.xacro (robot description, xacro)
@@ -29,4 +29,24 @@
 	    	</collision>
 	</link>
+	<link name="rear_right_wheel">
+		<visual>
+			<origin xyz="0 0 0" rpy="${PI/2} 0 0" />
+			<geometry>
+				<cylinder length="${wheel_width}" radius="${wheel_radius}"/>
+			</geometry>
+			<material name="Green" />
+		</visual>
+		<collision>
+			<origin xyz="0 0 0" rpy="${PI/2} 0 0" />
+			<geometry>
+				<cylinder length="${wheel_width}" radius="${wheel_radius}"/>
+			</geometry>
+		</collision>
+	</link>
+	<joint name="rear_right_wheel_to_rover_rear_right_wheel" type="fixed">
+		<origin xyz="0 0 0" rpy="0 0 0" />
+		<parent link="rear_right_wheel" />
+		<child link="rover_rear_right_wheel" />
+	</joint>
   	<joint name="rear_right_wheel_to_base" type="continuous">
 	    <origin xyz="-0.0600000000000001 -0.1135 -0.024" rpy="0 0 0" />

Commit message: base_link fixed

File: urdf/rover.xacro (robot description, xacro)
@@ -1,11 +1,11 @@
 <?xml version="1.0" encoding="utf-8"?>
 <robot name="rover" xmlns:xacro="http://www.ros.org/wiki/xacro">
-	<xacro:property name="clearance" value="0.074" />
+	<xacro:property name="clearance" value="0.07125" />
 	<xacro:property name="wheel_radius" value="0.0485"/>
-	<xacro:property name="wheel_separation_x" value="0.128"/>
-	<xacro:property name="wheel_separation_y" value="0.128"/>
+	<xacro:property name="wheel_separation_x" value="0.12"/>
+	<xacro:property name="wheel_separation_y" value="0.225"/>
 	<xacro:property name="wheel_width" value="0.0447"/>
 	<xacro:property name="PI" value="3.1415926"/>
-	<link name="base_link">
+	<link name="rover_base">
 		<inertial>
       			<origin xyz="0.00324310262857996 0.00100884866338095 0.00844749410443346" rpy="0 0 0" />
@@ -35,4 +35,17 @@
     		</collision>
   	</link>
+	<link name="base_link">
+		<visual>
+			<origin xyz="0 0 0" rpy="0 0 0" />
+			<geometry>
+				<sphere radius="0.001" />
+			</geometry>
+		</visual>
+	</link>
+	<joint name="base_link_to_rover_base" type="fixed">
+		<origin xyz="0 0 0" rpy="0 0 0" />
+		<parent link="base_link" />
+		<child link="rover_base" />
+	</joint>
 	<link name="base_footprint">
 		<visual>

Commit message: clearance value corrected

File: urdf/rover.xacro (robot description, xacro)
@@ -1,5 +1,5 @@
 <?xml version="1.0" encoding="utf-8"?>
 <robot name="rover" xmlns:xacro="http://www.ros.org/wiki/xacro">
-	<xacro:property name="clearance" value="0.07125" />
+	<xacro:property name="clearance" value="0.074" />
 	<xacro:property name="wheel_radius" value="0.0485"/>
 	<xacro:property name="wheel_separation_x" value="0.12"/>

Commit message: rplidar exported to urdf

File: urdf/rover.xacro (robot description, xacro)
@@ -9,6 +9,6 @@
 	<link name="rover_base">
 		<inertial>
-      			<origin xyz="0.00324310262857996 0.00100884866338095 0.00844749410443346" rpy="0 0 0" />
-      			<mass value="0.806772651118244" />
+      			<origin xyz="0.00149209044732787 -0.000940550840598575 0.00638419893745637" rpy="0 0 0" />
+      			<mass value="0.841151400832089" />
       			<inertia
       				ixx="0.00119589539435053"

File: urdf/rover_front_left_wheel.xacro (robot description, xacro)
@@ -50,8 +50,8 @@
 	</joint>
 	<joint name="front_left_wheel_to_base" type="continuous">
-	    	<origin xyz="0.0599999999999999 0.1135 -0.024" rpy="0 0 0" />
-	    	<parent link="rover_base" />
-	    	<child link="front_left_wheel" />
-	    	<axis xyz="0 -1 0" />
+	    <origin xyz="0.0599999999999999 0.1135 -0.024" rpy="0 0 0" />
+	    <parent link="rover_base" />
+	    <child link="front_left_wheel" />
+	    <axis xyz="0 1 0" />
 	</joint>
 </robot>

File: urdf/rover_rear_left_wheel.xacro (robot description, xacro)
@@ -50,8 +50,8 @@
 	</joint>
 	<joint name="rear_left_wheel_to_base" type="continuous">
-	    	<origin xyz="-0.0599999999999999 0.1135 -0.0240000000000001" rpy="0 0 0" />
-	    	<parent link="rover_base" />
-	    	<child link="rear_left_wheel" />
-	    	<axis xyz="0 -1 0" />
+	    <origin xyz="-0.0599999999999999 0.1135 -0.0240000000000001" rpy="0 0 0" />
+	    <parent link="rover_base" />
+	    <child link="rear_left_wheel" />
+	    <axis xyz="0 1 0" />
 	</joint>
 </robot>

Commit message: add realsense

File: urdf/rover.xacro (robot description, xacro)
@@ -70,3 +70,8 @@
 	<xacro:include filename="$(find rover_description)/urdf/rover_rear_right_wheel.xacro" />
 	<xacro:include filename="$(find rover_description)/urdf/rover_sensors.xacro" />
+	<xacro:include filename="$(find realsense2_description)/urdf/_d435i.urdf.xacro"/>
+	<xacro:sensor_d435i parent="base_link" name="d435i_camera">
+    		<origin xyz="0.0787368935630146 0.00750000000000009 0.0593651895857441"
+      		rpy="0 -0.261799387799143 0" />
+  	</xacro:sensor_d435i>
 </robot>

File: urdf/rover_sensors.xacro (robot description, xacro)
@@ -28,5 +28,5 @@
         name="">
         <color
-          rgba="0.752941176470588 0.752941176470588 0.752941176470588 1" />
+          rgba="0.2 0.2 0.2 1" />
       </material>
     </visual>
